Commit message: Add files via upload
Added counter
Added collisions
Added joint_counter

File: robo-arm-description/urdf/env_demo.urdf (robot description, URDF)
Before this commit: robot my_robot, 12 links, 11 joints
Links:
- added link counter; collision box size=0.5 0.2 0.01; visual box size=0.5 0.2 0.01
- link base_link: geometry collision box size=1 1 0.02; visual box size=1 1 0.02
- link x1_shelf_btm_link: geometry collision box size=0.5 0.2 0.01; visual box size=0.5 0.2 0.01
- link x1_shelf_top_link: geometry collision box size=0.5 0.2 0.01; visual box size=0.5 0.2 0.01
- link x1_wall_link: geometry collision box size=1 0.8 0.02; visual box size=1 0.8 0.02
- link x2_shelf_btm_link: geometry collision box size=0.5 0.2 0.01; visual box size=0.5 0.2 0.01
- link x2_shelf_top_link: geometry collision box size=0.5 0.2 0.01; visual box size=0.5 0.2 0.01
- link x2_wall_link: geometry collision box size=1 0.8 0.02; visual box size=1 0.8 0.02
- link y1_shelf_btm_link: geometry collision box size=0.5 0.2 0.01; visual box size=0.5 0.2 0.01
- link y1_shelf_top_link: geometry collision box size=0.5 0.2 0.01; visual box size=0.5 0.2 0.01
- link y1_wall_link: geometry collision box size=0.8 1 0.02; visual box size=0.8 1 0.02
- link y2_wall_link: geometry collision box size=0.3 1 0.02; visual box size=0.3 1 0.02
- link y2_wall_top_link: geometry collision box size=0.3 1 0.02; visual box size=0.3 1 0.02
Joints:
- added joint joint_counter: type fixed, parent y2_wall_link, child counter, origin xyz=0 0 0 rpy=0 0 0, axis 0 0 0
