Commit message: Added robo-arm-gazebo

File: robo-arm-description/urdf/panda.urdf (robot description, URDF)
Before this commit: robot panda, 12 links, 11 joints
Links:
- link panda_hand: mass None -> 1; geometry collision mesh filename=file://$(find robo-arm-description)/meshes/collision/hand.s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; visual mesh filename=file://$(find robo-arm-description)/meshes/visual/hand.dae
- link panda_leftfinger: mass None -> 1; geometry collision mesh filename=file://$(find robo-arm-description)/meshes/collision/finger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; visual mesh filename=file://$(find robo-arm-description)/meshes/visual/finger.dae
- link panda_link0: mass None -> 1; geometry collision mesh filename=file://$(find robo-arm-description)/meshes/collision/link0.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; visual mesh filename=file://$(find robo-arm-description)/share/robo-arm-descript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
- link panda_link1: mass None -> 1; geometry collision mesh filename=file://$(find robo-arm-description)/meshes/collision/link1.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; visual mesh filename=file://$(find robo-arm-description)/meshes/visual/link1.dae
- link panda_link2: mass None -> 1; geometry collision mesh filename=file://$(find robo-arm-description)/meshes/collision/link2.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; visual mesh filename=file://$(find robo-arm-description)/meshes/visual/link2.dae
- link panda_link3: mass None -> 1; geometry collision mesh filename=file://$(find robo-arm-description)/meshes/collision/link3.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; visual mesh filename=file://$(find robo-arm-description)/meshes/visual/link3.dae
- link panda_link4: mass None -> 1; geometry collision mesh filename=file://$(find robo-arm-description)/meshes/collision/link4.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; visual mesh filename=file://$(find robo-arm-description)/meshes/visual/link4.dae
- link panda_link5: mass None -> 1; geometry collision mesh filename=file://$(find robo-arm-description)/meshes/collision/link5.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; visual mesh filename=file://$(find robo-arm-description)/meshes/visual/link5.dae
- link panda_link6: mass None -> 1; geometry collision mesh filename=file://$(find robo-arm-description)/meshes/collision/link6.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; visual mesh filename=file://$(find robo-arm-description)/meshes/visual/link6.dae
- link panda_link7: geometry collision mesh filename=file://$(find robo-arm-description)/meshes/collision/link7.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; visual mesh filename=file://$(find robo-arm-description)/meshes/visual/link7.dae
- link panda_rightfinger: mass None -> 1; geometry collision mesh filename=file://$(find robo-arm-description)/meshes/collision/finger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; visual mesh filename=file://$(find robo-arm-description)/meshes/visual/finger.dae

Commit message: Update

File: robo-arm-description/urdf/panda.urdf (robot description, URDF)
Before this commit: robot panda, 12 links, 11 joints
Links:
- link panda_hand: geometry collision mesh filename=/home/cryptic/robo_arm_ws/src/robo-arm-ROS2/robo-arm-descri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; visual mesh filename=/home/cryptic/robo_arm_ws/src/robo-arm-ROS2/robo-arm-descri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
- link panda_leftfinger: geometry collision mesh filename=/home/cryptic/robo_arm_ws/src/robo-arm-ROS2/robo-arm-descri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; visual mesh filename=/home/cryptic/robo_arm_ws/src/robo-arm-ROS2/robo-arm-descri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
- link panda_link0: geometry collision mesh filename=/home/cryptic/robo_arm_ws/src/robo-arm-ROS2/robo-arm-descri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; visual mesh filename=/home/cryptic/robo_arm_ws/src/robo-arm-ROS2/robo-arm-descri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
- link panda_link1: geometry collision mesh filename=/home/cryptic/robo_arm_ws/src/robo-arm-ROS2/robo-arm-descri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; visual mesh filename=/home/cryptic/robo_arm_ws/src/robo-arm-ROS2/robo-arm-descri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
- link panda_link2: geometry collision mesh filename=/home/cryptic/robo_arm_ws/src/robo-arm-ROS2/robo-arm-descri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; visual mesh filename=/home/cryptic/robo_arm_ws/src/robo-arm-ROS2/robo-arm-descri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
- link panda_link3: geometry collision mesh filename=/home/cryptic/robo_arm_ws/src/robo-arm-ROS2/robo-arm-descri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; visual mesh filename=/home/cryptic/robo_arm_ws/src/robo-arm-ROS2/robo-arm-descri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
- link panda_link4: geometry collision mesh filename=/home/cryptic/robo_arm_ws/src/robo-arm-ROS2/robo-arm-descri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; visual mesh filename=/home/cryptic/robo_arm_ws/src/robo-arm-ROS2/robo-arm-descri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
- link panda_link5: geometry collision mesh filename=/home/cryptic/robo_arm_ws/src/robo-arm-ROS2/robo-arm-descri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; visual mesh filename=/home/cryptic/robo_arm_ws/src/robo-arm-ROS2/robo-arm-descri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
- link panda_link6: geometry collision mesh filename=/home/cryptic/robo_arm_ws/src/robo-arm-ROS2/robo-arm-descri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; visual mesh filename=/home/cryptic/robo_arm_ws/src/robo-arm-ROS2/robo-arm-descri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
- link panda_link7: geometry collision mesh filename=/home/cryptic/robo_arm_ws/src/robo-arm-ROS2/robo-arm-descri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; visual mesh filename=/home/cryptic/robo_arm_ws/src/robo-arm-ROS2/robo-arm-descri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
- link panda_rightfinger: geometry collision mesh filename=/home/cryptic/robo_arm_ws/src/robo-arm-ROS2/robo-arm-descri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; visual mesh filename=/home/cryptic/robo_arm_ws/src/robo-arm-ROS2/robo-arm-descri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

Commit message: Update

File: robo-arm-description/urdf/panda.urdf (robot description, URDF)
Before this commit: robot panda, 12 links, 11 joints
Links:
- link panda_hand: geometry collision mesh filename=package://robo-arm-description/meshes/collision/hand.stl; visual mesh filename=package://robo-arm-description/meshes/visual/hand.dae
- link panda_leftfinger: geometry collision mesh filename=package://robo-arm-description/meshes/collision/finger.stl; visual mesh filename=package://robo-arm-description/meshes/visual/finger.dae
- link panda_link0: geometry collision mesh filename=package://robo-arm-description/meshes/collision/link0.stl; visual mesh filename=package://robo-arm-description/meshes/visual/link0.dae
- link panda_link1: geometry collision mesh filename=package://robo-arm-description/meshes/collision/link1.stl; visual mesh filename=package://robo-arm-description/meshes/visual/link1.dae
- link panda_link2: geometry collision mesh filename=package://robo-arm-description/meshes/collision/link2.stl; visual mesh filename=package://robo-arm-description/meshes/visual/link2.dae
- link panda_link3: geometry collision mesh filename=package://robo-arm-description/meshes/collision/link3.stl; visual mesh filename=package://robo-arm-description/meshes/visual/link3.dae
- link panda_link4: geometry collision mesh filename=package://robo-arm-description/meshes/collision/link4.stl; visual mesh filename=package://robo-arm-description/meshes/visual/link4.dae
- link panda_link5: geometry collision mesh filename=package://robo-arm-description/meshes/collision/link5.stl; visual mesh filename=package://robo-arm-description/meshes/visual/link5.dae
- link panda_link6: geometry collision mesh filename=package://robo-arm-description/meshes/collision/link6.stl; visual mesh filename=package://robo-arm-description/meshes/visual/link6.dae
- link panda_link7: geometry collision mesh filename=package://robo-arm-description/meshes/collision/link7.stl; visual mesh filename=package://robo-arm-description/meshes/visual/link7.dae
- link panda_rightfinger: geometry collision mesh filename=package://robo-arm-description/meshes/collision/finger.stl; visual mesh filename=package://robo-arm-description/meshes/visual/finger.dae
