Commit message: Modified by Paul

File: robo-arm-gazebo/models/environment/book.urdf (robot description, URDF)
Before this commit: robot book, 1 links, 0 joints
Links:
- removed link book
- added link base_link, mass 0.5; collision box size=0.2 0.05 0.2; visual box size=0.2 0.05 0.2

Commit message: Modified by Paul

File: robo-arm-gazebo/models/environment/book.urdf (robot description, URDF)
Before this commit: robot book, 1 links, 0 joints
Links:
- added link base_footprint
- link base_link: geometry collision box size=0.12 0.04 0.15; visual box size=0.12 0.04 0.15
Joints:
- added joint base_footprint_joint: type fixed, parent base_footprint, child base_link
