Commit message: Add files via upload
double the size

File: robo-arm-gazebo/models/environment/bookshelf.urdf (robot description, URDF)
Before this commit: robot bookshelf, 13 links, 12 joints
Links:
- removed link x1_shelf_top_link
- removed link x2_shelf_top_link
- removed link y1_shelf_top_link
- link base_link: geometry collision box size=2 2 0.02; visual box size=2 2 0.02
- link counter: geometry collision box size=1 0.2 0.01; visual box size=1 0.2 0.01
- link x1_shelf_btm_link: geometry collision box size=1 0.2 0.01; visual box size=1 0.2 0.01
- link x1_wall_link: geometry collision box size=2 0.8 0.02; visual box size=2 0.8 0.02
- link x2_shelf_btm_link: geometry collision box size=1 0.2 0.01; visual box size=1 0.2 0.01
- link x2_wall_link: geometry collision box size=2 0.8 0.02; visual box size=2 0.8 0.02
- link y1_shelf_btm_link: geometry collision box size=1 0.2 0.01; visual box size=1 0.2 0.01
- link y1_wall_link: geometry collision box size=0.8 2 0.02; visual box size=0.8 2 0.02
- link y2_wall_link: geometry collision box size=0.3 1 0.02; visual box size=0.3 2 0.02
- link y2_wall_top_link: geometry collision box size=0.3 2 0.02; visual box size=0.3 2 0.02
Joints:
- removed joint joint_x1_shelf_top
- removed joint joint_x2_shelf_top
- removed joint joint_y1_shelf_top
- joint joint_x1_wall: origin xyz=0 0.51 0.41 rpy=0 0 0 -> xyz=0 1.01 0.41 rpy=0 0 0
- joint joint_x2_wall: origin xyz=0 -0.51 0.41 rpy=0 0 0 -> xyz=0 -1.01 0.41 rpy=0 0 0
- joint joint_y1_wall: origin xyz=0.51 0 0.41 rpy=0 0 0 -> xyz=1.01 0 0.41 rpy=0 0 0
- joint joint_y2_wall: origin xyz=-0.51 0 0.16 rpy=0 0 0 -> xyz=-1.01 0 0.16 rpy=0 0 0
- joint joint_y2_wall_top: origin xyz=-0.51 0 0.64 rpy=0 0 0 -> xyz=-1.01 0 0.64 rpy=0 0 0
